File: hardware/Source/nervous-ecg.kicad_sch (KiCad schematic)
At the start: 66 parts, among them J1 CONN RCP USB3.1 TYPEC 24P SMD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, J2 MOLEX 53048-0310, J3 CONN HEADER R/A 4POS 2.54MM, U1 RF TXRX MODULE BT TRACE ANT S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, U10 LIGHTPIPE PNL MT CONVEX 0.250", U11 LIGHTPIPE PNL MT CONVEX 0.250", U2 IC BATT CHG LI-ION 1CELL 16QFN, U3 IC BATT FUEL GAUGE LICOO2 12S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, U4 IC REG LINEAR 3.3V 200MA SOT2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, U5 IC ECG FRONT END 20LFCSP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

Commit message: fix : readjustment of decoupling capacitors positioning
Parts:
- BT1: value BATT LI-PO 3.7V 165MAH -> BATT LI-PO 3.7V 165MAH

Commit message: feat: bump to kicad 9.0.0
Parts:
- renumbered R43 to R28, R42 to R29
Changed lines of the file:
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@@
 (kicad_sch
-	(version 20231120)
+	(version 20250114)
 	(generator "eeschema")
-	(generator_version "8.0")
+	(generator_version "9.0")
 	(paper "A3")
 	(title_block
 		(title "NERVOUS - ECG Sensor")
-		(date "2024-05-02")
+		(date "2025-03-20")
 		(rev "1")
 		(comment 1 "Copyright (c) 2024 INSA Lyon, CNRS, INL UMR5270")
@@
 		(comment 4 "Authors : Bertrand Massot, Matthieu Mesnage, Hugo Buy")
 	)
+	(rectangle
+		(start 15.24 215.9)
+		(end 163.83 275.59)
+		(stroke
+			(width 0)
+			(type default)
+		)
+		(fill
+			(type none)
+		)
+	)
+	(rectangle
+		(start 13.97 16.51)
+		(end 231.14 100.33)
+		(stroke
+			(width 0)
+			(type default)
+		)
+		(fill
+			(type none)
+		)
+	)
+	(rectangle
+		(start 168.91 157.48)
+		(end 295.91 275.59)
+		(stroke
+			(width 0)
+			(type default)
+		)
+		(fill
+			(type none)
+		)
+	)
+	(rectangle
+		(start 313.69 143.51)
+		(end 375.92 172.72)
+		(stroke
+			(width 0)
+			(type default)
+		)
+		(fill
+			(type none)
+		)
+	)
+	(rectangle
+		(start 313.69 180.34)
+		(end 375.92 210.82)
+		(stroke
+			(width 0)
+			(type default)
+		)
+		(fill
+			(type none)
+		)
+	)
+	(rectangle
+		(start 26.67 118.11)
+		(end 152.4 189.23)
+		(stroke
+			(width 0)
+			(type default)
+		)
+		(fill
+			(type none)
+		)
+	)
+	(rectangle
+		(start 232.41 16.51)
+		(end 403.86 137.16)
+		(stroke
+			(width 0)
+			(type default)
+		)
+		(fill
+			(type none)
+		)
+	)
+	(text "RGB Led"
+		(exclude_from_sim no)
+		(at 374.65 172.72 0)
+		(effects
+			(font
+				(size 1.27 1.27)
+			)
+			(justify right bottom)
+		)
+	)
+	(text "Fuel Gauge"
+		(exclude_from_sim no)
+		(at 151.13 189.23 0)
+		(effects
+			(font
+				(size 1.27 1.27)
+			)
+			(justify right bottom)
+		)
+	)
+	(text "USB-C Connector and Battery Charger"
+		(exclude_from_sim no)
+		(at 229.87 100.33 0)
+		(effects
+			(font
+				(size 1.27 1.27)
+			)
+			(justify right bottom)
+		)
+	)
+	(text "ECG Frontend"
+		(exclude_from_sim no)
+		(at 294.64 275.59 0)
+		(effects
+			(font
+				(size 1.27 1.27)
+			)
+			(justify right bottom)
+		)
+	)
+	(text "SWD Connector"
+		(exclude_from_sim no)
+		(at 374.65 210.82 0)
+		(effects
+			(font
+				(size 1.27 1.27)
+			)
+			(justify right bottom)
+		)
+	)
+	(text "Microcontroller Unit"
+		(exclude_from_sim no)
+		(at 402.59 137.16 0)
+		(effects
+			(font
+				(size 1.27 1.27)
+			)
+			(justify right bottom)
+		)
+	)
+	(text "On-Off and Voltage Regulator"
+		(exclude_from_sim no)
+		(at 162.56 275.59 0)
+		(effects
+			(font
+				(size 1.27 1.27)
+			)
+			(justify right bottom)
+		)
+	)
+	(text_box "BQ24074 Configuration :\n\nRset = 5.93k  (Iset (155mA max) = 890 / Rset)\nRlim = 3.05k  (Ilim (500mA max) = 1525 / Rlim)\nDo not mount R5 if battery pack has 10k thermistor"
+		(exclude_from_sim no)
+		(at 97.79 30.48 0)
+		(size 55.88 12.7)
+		(margins 0.9525 0.9525 0.9525 0.9525)
+		(stroke
+			(width 0)
+			(type default)
+		)
+		(fill
+			(type none)
+		)
+		(effects
+			(font
+				(size 1.27 1.27)
+			)
+			(justify left top)
+		)
+	)
 	(junction
 		(at 275.59 243.84)
@@
 		)
 	)
-	(rectangle
-		(start 15.24 215.9)
-		(end 163.83 275.59)
-		(stroke
-			(width 0)
-			(type default)
-		)
-		(fill
-			(type none)
-		)
-	)
-	(rectangle
-		(start 13.97 16.51)
-		(end 231.14 100.33)
-		(stroke
-			(width 0)
-			(type default)
-		)
-		(fill
-			(type none)
-		)
-	)
-	(rectangle
-		(start 168.91 157.48)
-		(end 295.91 275.59)
-		(stroke
-			(width 0)
-			(type default)
-		)
-		(fill
-			(type none)
-		)
-	)
-	(rectangle
-		(start 313.69 143.51)
-		(end 375.92 172.72)
-		(stroke
-			(width 0)
-			(type default)
-		)
-		(fill
-			(type none)
-		)
-	)
-	(rectangle
-		(start 313.69 180.34)
-		(end 375.92 210.82)
-		(stroke
-			(width 0)
-			(type default)
-		)
-		(fill
-			(type none)
-		)
-	)
-	(rectangle
-		(start 26.67 118.11)
-		(end 152.4 189.23)
-		(stroke
-			(width 0)
-			(type default)
-		)
-		(fill
-			(type none)
-		)
-	)
-	(rectangle
-		(start 232.41 16.51)
-		(end 403.86 137.16)
-		(stroke
-			(width 0)
-			(type default)
-		)
-		(fill
-			(type none)
-		)
-	)
-	(text_box "BQ24074 Configuration :\n\nRset = 5.93k  (Iset (155mA max) = 890 / Rset)\nRlim = 3.05k  (Ilim (500mA max) = 1525 / Rlim)\nDo not mount R5 if battery pack has 10k thermistor"
-		(exclude_from_sim no)
-		(at 102.87 30.48 0)
-		(size 44.45 12.7)
-		(stroke
-			(width 0)
-			(type default)
-		)
-		(fill
-			(type none)
-		)
-		(effects
-			(font
-				(size 1.27 1.27)
-			)
-			(justify left top)
-		)
-	)
-	(text "RGB Led"
-		(exclude_from_sim no)
-		(at 374.65 172.72 0)
-		(effects
-			(font
-				(size 1.27 1.27)
-			)
-			(justify right bottom)
-		)
-	)
-	(text "Fuel Gauge"
-		(exclude_from_sim no)
-		(at 151.13 189.23 0)
-		(effects
-			(font
-				(size 1.27 1.27)
-			)
-			(justify right bottom)
-		)
-	)
-	(text "USB-C Connector and Battery Charger"
-		(exclude_from_sim no)
-		(at 229.87 100.33 0)
-		(effects
-			(font
-				(size 1.27 1.27)
-			)
-			(justify right bottom)
-		)
-	)
-	(text "ECG Frontend"
-		(exclude_from_sim no)
-		(at 294.64 275.59 0)
-		(effects
-			(font
-				(size 1.27 1.27)
-			)
-			(justify right bottom)
-		)
-	)
-	(text "SWD Connector"
-		(exclude_from_sim no)
-		(at 374.65 210.82 0)
-		(effects
-			(font
-				(size 1.27 1.27)
-			)
-			(justify right bottom)
-		)
-	)
-	(text "Microcontroller Unit"
-		(exclude_from_sim no)
-		(at 402.59 137.16 0)
-		(effects
-			(font
-				(size 1.27 1.27)
-			)
-			(justify right bottom)
-		)
-	)
-	(text "On-Off and Voltage Regulator"
-		(exclude_from_sim no)
-		(at 162.56 275.59 0)
-		(effects
-			(font
-				(size 1.27 1.27)
-			)
-			(justify right bottom)
-		)
-	)
 	(label "RA"
 		(at 184.15 195.58 0)
@@
 		(on_board yes)
 		(dnp no)
-		(property "Reference" "R43"
+		(property "Reference" "R28"
 			(at 20.32 68.58 0)
 			(effects
@@
 		(on_board yes)
 		(dnp no)
-		(property "Reference" "R42"
+		(property "Reference" "R29"
 			(at 29.21 68.58 0)
 			(effects
@@
 		)
 	)
+	(embedded_fonts no)
 )
